Commit message: 変更：livox_frameの指定にミスがあったため直した。点群がロボットに合わせて景色が動くことを確認

File: urdf/parts/mid360.urdf.xacro (robot description, xacro)
@@ -2,8 +2,8 @@
 <robot xmlns:xacro="http://www.ros.org/wiki/xacro">
   <xacro:macro name="mid360">
-    <link name="mid360_link"/>
+    <link name="livox_frame"/>
     <joint name="base_to_mid360_joint" type="fixed">
       <origin xyz="0.3 0 0.12" rpy="0 0.6109 0" />
-      <parent link="base_link"/> <child link="mid360_link"/>
+      <parent link="base_link"/> <child link="livox_frame"/>
     </joint>
   </xacro:macro>
